File: Hardware/KiCad5/CloudSmoker.sch (KiCad schematic (older format))
At the start: 8 parts, among them J1 Barrel_Jack, J2 Conn_01x03, U1 5V-3V3_StepDown_module_off-bo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

Commit message: Update schematic
Parts:
- J1: symbol CloudSmoker-rescue:Barrel_Jack -> Connector:Barrel_Jack_Switch
- J2: symbol CloudSmoker-rescue:Conn_01x03 -> Connector_Generic:Conn_01x03
- U1: symbol CloudSmoker-rescue:5V-3V3_StepDown_module_off-board -> cg_off-board:5V-3V3_StepDown_module_off-board
Changed lines of the file:
@@
 Sheet 1 4
 Title "CloudSmoker - Wifi enabled BBQ Temperature Monitor"
-Date "2017-09-14"
+Date "2021-01-01"
 Rev "1"
 Comp "Carl Greenstreet"
 Comment1 ""
-Comment2 ""
+Comment2 "Main (top) sheet"
 Comment3 ""
 Comment4 ""
 $EndDescr
 $Comp
-L CloudSmoker-rescue:Barrel_Jack J1
+L Connector:Barrel_Jack_Switch J1
 U 1 1 59B9C571
 P 1200 1250
 F 0 "J1" H 1200 1460 50  0000 C CNN
-F 1 "Barrel_Jack" H 1200 1075 50  0000 C CNN
+F 1 "Barrel_Jack" H 1200 1050 50  0000 C CNN
 F 2 "" H 1250 1210 50  0001 C CNN
 F 3 "" H 1250 1210 50  0001 C CNN
@@
 GND
 $Comp
-L CloudSmoker-rescue:Conn_01x03 J2
+L Connector_Generic:Conn_01x03 J2
 U 1 1 59DEBC06
 P 5600 1550
@@
 $EndComp
 $Comp
-L CloudSmoker-rescue:5V-3V3_StepDown_module_off-board U1
+L cg_off-board:5V-3V3_StepDown_module_off-board U1
 U 1 1 59DEBC0D
 P 4200 1550

Commit message: schematic updates
Parts:
- added D1: D_Schottky, symbol Device:D_Schottky
- C1: value C -> 22uF
Connections:
- net +3V3: now also C1.1, J2.1 (Pin_1), D1.1 (K)
- removed net +5V: C1.1, J1.1, J2.1 (Pin_1)
- new net: D1.2 (A), J1.1
Other:
- note added: "Reverse polarity protection\nMBRA130, BAT54, \nPMEG3020CEP or similar \nlow Vf drop diode\n"
- moved on the sheet: C1, C2, C3, J1, J2, L1, R1, U1
