File: Hardware/KiCad5/ESP8266-07.sch (KiCad schematic (older format))
At the start: 20 parts, among them J3 Conn_01x06, SW1 SW_Push, SW2 SW_Push, U2 ESP-07v2

Commit message: Update schematic
Parts:
- J3: symbol CloudSmoker-rescue:Conn_01x06 -> Connector_Generic:Conn_01x06
- SW1, SW2: symbol CloudSmoker-rescue:SW_Push -> Switch:SW_Push
- U2: symbol CloudSmoker-rescue:ESP-07v2 -> cg_modules:ESP-07v2
Changed lines of the file:
@@
 $EndDescr
 $Comp
-L CloudSmoker-rescue:ESP-07v2 U2
+L cg_modules:ESP-07v2 U2
 U 1 1 59BACA1D
 P 5700 3650
@@
 $EndComp
 $Comp
-L CloudSmoker-rescue:Conn_01x06 J3
+L Connector_Generic:Conn_01x06 J3
 U 1 1 59BACD0E
 P 9300 3550
@@
 $EndComp
 $Comp
-L CloudSmoker-rescue:SW_Push SW1
+L Switch:SW_Push SW1
 U 1 1 59BACFC1
 P 3450 3850
@@
 $EndComp
 $Comp
-L CloudSmoker-rescue:SW_Push SW2
+L Switch:SW_Push SW2
 U 1 1 59BAD014
 P 8500 4000
@@
 	8800 4150 8800 3450
 Wire Wire Line
-	6600 3450 9100 3450
+	6600 3450 8800 3450
 Connection ~ 6800 2700
 Wire Wire Line
@@
 	7400 3750 7400 3150
 Wire Wire Line
-	6600 3550 7600 3550
-Wire Wire Line
-	6600 3650 7750 3650
+	6600 3550 6800 3550
+Wire Wire Line
+	6600 3650 7000 3650
 Connection ~ 3450 4700
 Wire Wire Line
-	3450 4700 3450 4050
+	3450 4700 3450 4150
 Connection ~ 3450 3350
 Connection ~ 3450 2600
@@
 	3450 2600 3450 2850
 Wire Wire Line
-	3450 3150 3450 3650
+	3450 3150 3450 3350
 Connection ~ 3200 2600
 Wire Wire Line
@@
 	7200 3850 7200 3150
 Wire Wire Line
-	6600 3850 8150 3850
+	6600 3850 7200 3850
 Wire Wire Line
 	7200 2700 7200 2850
 Wire Wire Line
-	5700 2700 7400 2700
+	5700 2700 6800 2700
 Connection ~ 2850 4700
 Wire Wire Line
@@
 	2850 2600 2850 4000
 Wire Wire Line
-	9000 4600 5700 4600
-Connection ~ 2300 4700
+	9000 4600 8800 4600
 Wire Wire Line
 	2300 4200 2300 4700
-Connection ~ 2300 2600
 Wire Wire Line
 	2300 2600 2300 3900
 Wire Wire Line
-	2300 4700 5700 4700
-Wire Wire Line
-	9000 3750 9000 4600
+	2300 4700 2850 4700
+Wire Wire Line
+	9000 3750 9000 4000
 Wire Wire Line
 	9000 3750 9100 3750
@@
 	6600 3350 9100 3350
 Wire Wire Line
-	5700 4550 5700 4750
-Wire Wire Line
-	4250 3750 4800 3750
+	5700 4550 5700 4600
+Wire Wire Line
+	4250 3750 4400 3750
 Wire Wire Line
 	4250 3750 4250 2450
 Wire Wire Line
-	4050 3850 4800 3850
+	4050 3850 4200 3850
 Wire Wire Line
 	4050 3850 4050 2450
 Wire Wire Line
-	2300 2600 5700 2600
+	2300 2600 2850 2600
 Wire Wire Line
 	7600 3550 7600 2450
 Wire Wire Line
-	6600 3750 7950 3750
+	6600 3750 7400 3750
 Wire Wire Line
 	7750 3650 7750 2450
@@
 	3850 3950 3850 2450
 Wire Wire Line
-	5700 2550 5700 2750
+	5700 2550 5700 2600
 Connection ~ 5700 2700
 Connection ~ 5700 2600
@@
 Connection ~ 4400 4700
 Wire Wire Line
-	3450 3350 4800 3350
+	3450 3350 4500 3350
 Connection ~ 4500 3350
+Wire Wire Line
+	8800 3450 9100 3450
+Wire Wire Line
+	6800 2700 7000 2700
+Wire Wire Line
+	6800 3550 7600 3550
+Wire Wire Line
+	7000 2700 7200 2700
+Wire Wire Line
+	7000 3650 7750 3650
+Wire Wire Line
+	6600 4600 5700 4600
+Wire Wire Line
+	3450 4150 3450 4050
+Wire Wire Line
+	8800 4600 6600 4600
+Wire Wire Line
+	7400 3750 7900 3750
+Wire Wire Line
+	7200 2700 7400 2700
+Wire Wire Line
+	3450 4700 4200 4700
+Wire Wire Line
+	3450 3350 3450 3650
+Wire Wire Line
+	3450 2600 5700 2600
+Wire Wire Line
+	3200 2600 3450 2600
+Wire Wire Line
+	5700 4700 5700 4750
+Wire Wire Line
+	2850 4700 3450 4700
+Wire Wire Line
+	2850 2600 3200 2600
+Wire Wire Line
+	9000 4000 9000 4600
+Wire Wire Line
+	5700 4600 5700 4700
+Wire Wire Line
+	5700 2700 5700 2750
+Wire Wire Line
+	5700 2600 5700 2700
+Wire Wire Line
+	7900 3750 7950 3750
+Wire Wire Line
+	7200 3850 8150 3850
+Wire Wire Line
+	4400 3750 4800 3750
+Wire Wire Line
+	4200 3850 4800 3850
+Wire Wire Line
+	4200 4700 4400 4700
+Wire Wire Line
+	4400 4700 5700 4700
+Wire Wire Line
+	4500 3350 4800 3350
 $EndSCHEMATC

Commit message: schematic updates
Parts:
- renumbered D1 to D2, D2 to D3
Changed lines of the file:
@@
 $EndComp
 $Comp
-L power1:GND #PWR012
+L power1:GND #PWR09
 U 1 1 59BACAED
 P 5700 4750
-F 0 "#PWR012" H 5700 4500 50  0001 C CNN
+F 0 "#PWR09" H 5700 4500 50  0001 C CNN
 F 1 "GND" H 5700 4600 50  0000 C CNN
 F 2 "" H 5700 4750 50  0001 C CNN
@@
 $EndComp
 $Comp
-L power1:+3.3V #PWR013
+L power1:+3.3V #PWR08
 U 1 1 59BACB07
 P 5700 2550
-F 0 "#PWR013" H 5700 2400 50  0001 C CNN
+F 0 "#PWR08" H 5700 2400 50  0001 C CNN
 F 1 "+3.3V" H 5700 2690 50  0000 C CNN
 F 2 "" H 5700 2550 50  0001 C CNN
@@
 MUX
 $Comp
-L device:D_Zener D2
+L device:D_Zener D3
 U 1 1 59BB0CC7
 P 8800 4300
-F 0 "D2" H 8800 4400 50  0000 C CNN
+F 0 "D3" H 8800 4400 50  0000 C CNN
 F 1 "3.3V" H 8800 4200 50  0000 C CNN
 F 2 "" H 8800 4300 50  0001 C CNN
@@
 	0    1    1    0
 $EndComp
-Text Notes 4850 5800 0    60   ~ 0
+Text Notes 5000 5550 0    60   ~ 0
 okay to leave unused GPIO pins floating; careful with others
 $Comp
@@
 	1    0    0    -1
 $EndComp
-Text Notes 4850 6050 0    60   ~ 0
+Text Notes 5000 5800 0    60   ~ 0
 GPIO4/GPIO5, GPIO12, 13, 14 => General purpose pins\nGPIO16 needed for deep sleep
 $Comp
@@
 $EndComp
 $Comp
-L device:D_Schottky D1
+L device:D_Schottky D2
 U 1 1 59BB5CEA
 P 4500 3500
-F 0 "D1" H 4500 3600 50  0000 C CNN
+F 0 "D2" H 4500 3600 50  0000 C CNN
 F 1 "D_Schottky" H 4500 3400 50  0000 C CNN
 F 2 "" H 4500 3500 50  0001 C CNN
@@
 	0    -1   -1   0
 $EndComp
-Text Notes 800  7500 0    60   ~ 0
+Text Notes 900  6650 0    60   ~ 0
 Schottky signal diode or 330 to 1K ohm resistor required between GPIO16 and REST pins\nGPIO16 is ony pin belonging to RTC (real time clock) module.  During deep sleep, GPIO16 pin is high.  \nWhen RTC triggers wake-up, it drives GPIO16 pin low, which also drives REST pin low, tirggering reset\n
 Text HLabel 4250 2450 1    60   Output ~ 0
@@
 Text HLabel 4050 2450 1    60   Output ~ 0
 CTL-B
-Text Notes 800  7200 0    60   ~ 12
+Text Notes 900  6300 0    60   ~ 12
 Deep Sleep
 Text HLabel 3850 2450 1    60   Input ~ 0
@@
 Text Notes 2100 3750 0    39   ~ 0
 Stabilise power rail
-Text Notes 1050 6000 0    60   ~ 0
+Text Notes 1200 5750 0    60   ~ 0
 GPIO4/GPIO5, GPIO12, 13, 14 => General purpose pins\nGPIO16 needed for deep sleep
 Text Notes 6250 2550 0    39   ~ 0
