File: Hardware/KiCad5/LCD.sch (KiCad schematic (older format))
At the start: 5 parts, among them J6 Conn_01x04, J7 Conn_01x05, SW3 Rotary_Encoder_Switch_off-boa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, U5 2CH_I2C_Logic_Level_Convertor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, U6 LCD_16x2_I2C_OffBoard

Commit message: schematic updates
Parts:
- J6: symbol CloudSmoker-rescue:Conn_01x04 -> Connector_Generic:Conn_01x04
- J7: symbol CloudSmoker-rescue:Conn_01x05 -> Connector_Generic:Conn_01x05
- SW3: symbol CloudSmoker-rescue:Rotary_Encoder_Switch_off-board -> cg_off-board:Rotary_Encoder_Switch_off-board
- U5: symbol CloudSmoker-rescue:2CH_I2C_Logic_Level_Convertor_Bidirectional -> cg_modules:2CH_I2C_Logic_Level_Convertor_Bidirectional
- U6: symbol CloudSmoker-rescue:LCD_16x2_I2C_OffBoard -> cg_display:LCD_16x2_I2C_OffBoard
Changed lines of the file:
@@
 $EndDescr
 $Comp
-L CloudSmoker-rescue:Conn_01x04 J6
+L Connector_Generic:Conn_01x04 J6
 U 1 1 59D724D0
 P 5200 3250
@@
 $EndComp
 $Comp
-L CloudSmoker-rescue:2CH_I2C_Logic_Level_Convertor_Bidirectional U5
+L cg_modules:2CH_I2C_Logic_Level_Convertor_Bidirectional U5
 U 1 1 59D72818
 P 3350 3200
@@
 Dupont wires to off-Board LCD\n(Mounted to enclosure window)
 $Comp
-L power1:+3.3V #PWR028
+L power1:+3.3V #PWR030
 U 1 1 59D72B2B
 P 3250 2700
-F 0 "#PWR028" H 3250 2550 50  0001 C CNN
+F 0 "#PWR030" H 3250 2550 50  0001 C CNN
 F 1 "+3.3V" H 3250 2840 50  0000 C CNN
 F 2 "" H 3250 2700 50  0001 C CNN
@@
 $EndComp
 $Comp
-L power1:+5V #PWR029
+L power1:+5V #PWR032
 U 1 1 59D72B4E
 P 3450 2700
-F 0 "#PWR029" H 3450 2550 50  0001 C CNN
+F 0 "#PWR032" H 3450 2550 50  0001 C CNN
 F 1 "+5V" H 3450 2840 50  0000 C CNN
 F 2 "" H 3450 2700 50  0001 C CNN
@@
 $EndComp
 $Comp
-L power1:GND #PWR030
+L power1:GND #PWR031
 U 1 1 59D72B81
 P 3250 3700
-F 0 "#PWR030" H 3250 3450 50  0001 C CNN
+F 0 "#PWR031" H 3250 3450 50  0001 C CNN
 F 1 "GND" H 3250 3550 50  0000 C CNN
 F 2 "" H 3250 3700 50  0001 C CNN
@@
 $EndComp
 $Comp
-L power1:GND #PWR031
+L power1:GND #PWR033
 U 1 1 59D72B9C
 P 3450 3700
-F 0 "#PWR031" H 3450 3450 50  0001 C CNN
+F 0 "#PWR033" H 3450 3450 50  0001 C CNN
 F 1 "GND" H 3450 3550 50  0000 C CNN
 F 2 "" H 3450 3700 50  0001 C CNN
@@
 SDA
 $Comp
-L CloudSmoker-rescue:LCD_16x2_I2C_OffBoard U6
+L cg_display:LCD_16x2_I2C_OffBoard U6
 U 1 1 59D80FE1
 P 7600 3250
@@
 	1    0    0    -1
 $EndComp
-Wire Notes Line
-	6350 2300 6350 4650
 Wire Notes Line
 	6350 4650 8950 4650
@@
 	5400 4400 6750 4400
 $Comp
-L CloudSmoker-rescue:Rotary_Encoder_Switch_off-board SW3
+L cg_off-board:Rotary_Encoder_Switch_off-board SW3
 U 1 1 59DC4E10
 P 7600 4250
@@
 $EndComp
 $Comp
-L CloudSmoker-rescue:Conn_01x05 J7
+L Connector_Generic:Conn_01x05 J7
 U 1 1 59DC4E88
 P 5200 4300
@@
 	1    0    0    -1
 $EndComp
-Wire Notes Line
-	6350 2400 6350 4750
 Wire Notes Line
 	5400 4500 6750 4500
@@
 Text Notes 8000 4200 0    39   ~ 0
 Solder two 0.1uF caps directly \nbetween encoder pins A-C \nand B-C (where C = GND).  \nAlso, 4-5 where 5=GND
+Wire Notes Line
+	6350 2300 6350 4750
 $EndSCHEMATC
